File: microbit_nrf54l20.kicad_sch (KiCad schematic)
At the start: 41 parts, among them J1 USB_Micro_B, J2 EDGE_CONNECTOR, J3 BAT_2xAAA, SW1 BTN_A, SW2 BTN_B, SW3 RESET, U1 nRF54L20, U2 LSM303C, U3 AP2112K-3.3, Y1 32MHz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

Commit message: Update symbols
Connections:
- net P10 is gone; now on net XL2: U1.49 (P1.21)
- net P11 is gone; now on net P16: U1.50 (P1.24)
- net +3V3: now also L1.2, U1.42 (VDD), U1.6 (VDD); no longer U1.1 (VDD), U1.2 (VDDH), U1.3 (VDD)
- net ACC_INT1: now also U1.12 (P1.02); no longer U1.34 (P1.09)
- net ACC_INT2: now also U1.13 (P1.03); no longer U1.35 (P1.10)
- net BTN_A: now also U1.7 (P1.29); no longer U1.30 (P1.05)
- net BTN_B: now also U1.8 (P1.30); no longer U1.31 (P1.06)
- net COL1: now also U1.14 (P1.04); no longer U1.25 (P1.00)
- net COL2: now also U1.15 (P1.05); no longer U1.26 (P1.01)
- net COL3: now also U1.16 (P1.06); no longer U1.27 (P1.02)
- net COL4: now also U1.22 (P1.07); no longer U1.28 (P1.03)
- net COL5: now also U1.23 (P1.08); no longer U1.29 (P1.04)
- net GND: now also U1.35 (VSS), U1.45 (VSS); no longer U1.19 (VSS), U1.52 (VSS)
- net MIC_OUT: now also U1.10 (P1.00); no longer U1.36 (P1.11)
- net MIC_RUN: now also U1.11 (P1.01); no longer U1.37 (P1.12)
- net P0: now also U1.1 (P2.01); no longer U1.39 (P1.14)
- net P1: now also U1.2 (P2.02); no longer U1.40 (P1.15)
- net P12: now also U1.39 (P1.15); no longer U1.44 (P2.03)
- net P13: now also U1.40 (P1.16); no longer U1.45 (P2.04)
- net P14: now also U1.41 (P1.18); no longer U1.46 (P2.05)
- net P16: no longer U1.48 (P2.07)
- net P2: now also U1.3 (P2.03); no longer U1.41 (P2.00)
- net P8: now also U1.4 (P2.04); no longer U1.42 (P2.01)
- net P9: now also U1.5 (P2.05); no longer U1.43 (P2.02)
- net RF_ANT: now also U1.34 (ANT); no longer U1.13 (ANT)
- net ROW1: now also U1.24 (P1.09); no longer U1.20 (P0.00)
- net ROW2: now also U1.25 (P0.03); no longer U1.21 (P0.01)
- net ROW3: now also U1.26 (P0.04); no longer U1.22 (P0.02)
- net ROW4: now also U1.27 (P0.06); no longer U1.23 (P0.03)
- net ROW5: now also U1.28 (P0.07); no longer U1.24 (P0.04)
- net SCL: now also U1.30 (P0.09); no longer U1.33 (P1.08)
- net SDA: now also U1.29 (P0.08); no longer U1.32 (P1.07)
- net SPK: now also U1.9 (P1.31); no longer U1.38 (P1.13)
- net SWDCLK: now also U1.31 (SWDCLK); no longer U1.15 (SWDCLK)
- net SWDIO: now also U1.32 (SWDIO); no longer U1.14 (SWDIO)
- net USB_DM: now also U1.20 (D-); no longer U1.18 (USB_DM)
- net USB_DP: now also U1.19 (D+); no longer U1.17 (USB_DP)
- net VBUS: now also U1.17 (VBUS)
- net XC1: now also U1.37 (XC1); no longer U1.9 (XC1)
- net XC2: now also U1.38 (XC2); no longer U1.10 (XC2)
- net XL1: now also U1.48 (P1.20); no longer U1.11 (XL1)
- net XL2: no longer U1.12 (XL2)
- net nRESET: now also U1.33 (nRESET); no longer U1.16 (nRESET)
- net DCDC_L1 renamed DCC
- net DCC: now also U1.43 (DCC); no longer U1.7 (DCDCL1)
- removed net DCDC_L2: L1.2, U1.8 (DCDCL2)
- net DEC1 renamed DECD
- net DECD: now also U1.44 (DECD); no longer U1.4 (DEC1)
- net DEC4 renamed DECA
- net DECA: now also U1.36 (DECRF), U1.46 (DECA); no longer U1.5 (DEC4)
- net DECRF renamed DECUSB
- net DECUSB: now also U1.18 (DECUSB); no longer U1.6 (DECRF)
- new net TXRTUNE: U1.21 (TXRTUNE)
