File: md_nrf54l20.kicad_pcb (KiCad board)
At the start: 2 copper layers, 0 parts

Commit message: Update layout
Parts:
- added C1: 10uF, Capacitor_SMD:C_0201_0603Metric, F.Cu at (142.3, 96.8)
- added C3: 100nF, Capacitor_SMD:C_0201_0603Metric, F.Cu at (142.3, 98.5)
- added C4: 100nF, Capacitor_SMD:C_0201_0603Metric, F.Cu at (142.3, 100.2)
- added C5: 100nF, Capacitor_SMD:C_0201_0603Metric, F.Cu at (142.3, 102.0)
- added J1: USB_C_Receptacle_USB2.0_16P, Connector_USB:USB_C_Receptacle_G-Switch_GT-USB-7010ASV, F.Cu at (149.2, 85.2)
- added U1: nRF54L20, md_nrf54l20:QFN-52-1EP_6x6mm_P0.4mm_EP4.7x4.7mm, F.Cu at (149.1, 101.9)
Other:
- board outline added: 51.6 x 42 mm
