File: md_nrf54l20.kicad_sch (KiCad schematic)
At the start: 41 parts, among them J1 USB_Micro_B, J2 EDGE_CONNECTOR, J3 BAT_2xAAA, SW1 BTN_A, SW2 BTN_B, SW3 RESET, U1 nRF54L20, U2 LSM303C, U3 AP2112K-3.3, Y1 32MHz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

Commit message: Update layout
Parts:
- removed ANT1: 2.4GHz, RF_Antenna:Johanson_2450AT18x100, symbol Device:Antenna
- removed C10, C7, C8, C9: 12pF, Capacitor_SMD:C_0402_1005Metric, symbol Device:C
- removed C11: 1.5pF, Capacitor_SMD:C_0402_1005Metric, symbol Device:C
- removed C12: 1.0pF, Capacitor_SMD:C_0402_1005Metric, symbol Device:C
- removed C13, C14, C15, C16, C17, C18, C21, C22: 100nF, Capacitor_SMD:C_0402_1005Metric, symbol Device:C
- removed C19: 1uF, Capacitor_SMD:C_0402_1005Metric, symbol Device:C
- removed C20: 4.7uF, Capacitor_SMD:C_0603_1608Metric, symbol Device:C
- removed C4, C5: 10uF, Capacitor_SMD:C_0805_2012Metric, symbol Device:C
- removed C6: 1uF, Capacitor_SMD:C_0603_1608Metric, symbol Device:C
- removed D26: PWR, LED_SMD:LED_0603_1608Metric, symbol Device:LED
- removed D27: BAT_OR, Diode_SMD:D_SOD-123, symbol Device:D_Schottky
- removed J1: USB_Micro_B, Connector_USB:USB_Micro-B_Molex-105017-0001, symbol Connector:USB_B_Micro
- removed J2: EDGE_CONNECTOR, Connector_PinHeader_2.54mm:PinHeader_1x25_P2.54mm_Vertical, symbol Connector_Generic:Conn_01x25
- removed J3: BAT_2xAAA, Connector_JST:JST_PH_S2B-PH-K_1x02_P2.00mm_Horizontal, symbol Connector_Generic:Conn_01x02
- removed L1: 10uH, Inductor_SMD:L_0603_1608Metric, symbol Device:L
- removed L2: 3.9nH, Inductor_SMD:L_0402_1005Metric, symbol Device:L
- removed LS1: SPEAKER, Buzzer_Beeper:Buzzer_Murata_PKLCS1212E, symbol Device:Buzzer
- removed MK1: MEMS_MIC, Sensor_Audio:CUI_CMC-4013-SMT, symbol Device:Microphone
- removed R10: 220, Resistor_SMD:R_0402_1005Metric, symbol Device:R
- removed R11: 10k, Resistor_SMD:R_0402_1005Metric, symbol Device:R
- removed R12, R13: 4.7k, Resistor_SMD:R_0402_1005Metric, symbol Device:R
- removed SW1: BTN_A, Button_Switch_SMD:SW_Push_1P1T_NO_CK_KMR2, symbol Switch:SW_Push
- removed SW2: BTN_B, Button_Switch_SMD:SW_Push_1P1T_NO_CK_KMR2, symbol Switch:SW_Push
- removed SW3: RESET, Button_Switch_SMD:SW_Push_1P1T_NO_CK_KMR2, symbol Switch:SW_Push
- removed U2: LSM303C, Package_LGA:LGA-12_2x2mm_P0.5mm, symbol Sensor_Motion:LSM303C
- removed U3: AP2112K-3.3, Package_TO_SOT_SMD:SOT-23-5, symbol Regulator_Linear:AP2112K-3.3
- removed Y1: 32MHz, Crystal:Crystal_SMD_3225-4Pin_3.2x2.5mm, symbol Device:Crystal_GND24
- removed Y2: 32.768kHz, Crystal:Crystal_SMD_3215-2Pin_3.2x1.5mm, symbol Device:Crystal
- added C1: 10uF, Capacitor_SMD:C_0201_0603Metric, symbol Device:C_Small
- added C3, C4, C5: 100nF, Capacitor_SMD:C_0201_0603Metric, symbol Device:C_Small
- added J1: USB_C_Receptacle_USB2.0_16P, Connector_USB:USB_C_Receptacle_G-Switch_GT-USB-7010ASV, symbol Connector:USB_C_Receptacle_USB2.0_16P
Connections:
- net VBUS is gone; now on net +3.3V: U1.17 (VBUS)
- net GND: now also C1.2, C3.2, C4.2, C5.2
- net P8: no longer U1.4 (P2.04)
- net P9: no longer U1.5 (P2.05)
- net +3V3 renamed +3.3V
- net +3.3V: now also C1.1, C3.1, C4.1, C5.1
- net ACC_INT1: no longer names the net of U1.12 (P1.02)
- net ACC_INT2: no longer names the net of U1.13 (P1.03)
- net BTN_A: no longer names the net of U1.7 (P1.29)
- net BTN_B: no longer names the net of U1.8 (P1.30)
- net COL1: no longer names the net of U1.14 (P1.04)
- net COL2: no longer names the net of U1.15 (P1.05)
- net COL3: no longer names the net of U1.16 (P1.06)
- net COL4: no longer names the net of U1.22 (P1.07)
- net COL5: no longer names the net of U1.23 (P1.08)
- net DCC: no longer names the net of U1.43 (DCC)
- net DECA: no longer names the net of U1.36 (DECRF)
- net DECA: no longer U1.46 (DECA)
- net DECD: no longer names the net of U1.44 (DECD)
- net DECUSB: no longer names the net of U1.18 (DECUSB)
- net MIC_OUT: no longer names the net of U1.10 (P1.00)
- net MIC_RUN: no longer names the net of U1.11 (P1.01)
- net P0: no longer names the net of U1.1 (P2.01)
- net P1: no longer names the net of U1.2 (P2.02)
- net P12: no longer names the net of U1.39 (P1.15)
- net P13: no longer names the net of U1.40 (P1.16)
- net P14: no longer names the net of U1.41 (P1.18)
- net P15: no longer names the net of U1.47 (P1.19)
- net P16: no longer names the net of U1.50 (P1.24)
- net P2: no longer names the net of U1.3 (P2.03)
- net RF_ANT: no longer names the net of U1.34 (ANT)
- net ROW1: no longer names the net of U1.24 (P1.09)
- net ROW2: no longer names the net of U1.25 (P0.03)
- net ROW3: no longer names the net of U1.26 (P0.04)
- net ROW4: no longer names the net of U1.27 (P0.06)
- net ROW5: no longer names the net of U1.28 (P0.07)
- net SCL: no longer names the net of U1.30 (P0.09)
- net SDA: no longer names the net of U1.29 (P0.08)
- net SPK: no longer names the net of U1.9 (P1.31)
- net SWDCLK: no longer names the net of U1.31 (SWDCLK)
- net SWDIO: no longer names the net of U1.32 (SWDIO)
- net TXRTUNE: no longer names the net of U1.21 (TXRTUNE)
- net USB_DM: no longer names the net of U1.20 (USB_D-)
- net USB_DP: no longer names the net of U1.19 (USB_D+)
- net XC1: no longer names the net of U1.37 (XC1)
- net XC2: no longer names the net of U1.38 (XC2)
- net XL1: no longer names the net of U1.48 (P1.20)
- net XL2: no longer names the net of U1.49 (P1.21)
- net nRESET: no longer names the net of U1.33 (nRESET)
- new net: J1.A1 (GND), J1.A12 (GND), J1.B1 (GND), J1.B12 (GND)
- new net: J1.A4 (VBUS), J1.A9 (VBUS), J1.B4 (VBUS), J1.B9 (VBUS)
Other:
- note added: "EDGE"
- moved on the sheet: U1
